File: test_boards/10CL006YE144C8G/10CL006YE144C8G.kicad_pcb (KiCad board)
At the start: 2 copper layers, 82 parts, among them IC1 10CL006YE144C8G, J1 CL_JTAG, U1 W25Q128JVS, Y1 SG-7050CAN

Commit message: Полный рефакторинг. Все тесты собраны вместе. Проверены
Parts:
- moved C1 7.67 mm to (166.5, 79.2), turned to 0 degrees
Changed lines of the file:
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@@
 	(footprint "Capacitor_SMD:C_0603_1608Metric_Pad1.08x0.95mm_HandSolder"
 		(layer "F.Cu")
-		(at 159.54 76 90)
+		(at 166.515 79.195)
 		(descr "Capacitor SMD 0603 (1608 Metric), square (rectangular) end terminal, IPC-7351 nominal with elongated pad for handsoldering. (Body size source: IPC-SM-782 page 76, https://www.pcb-3d.com/wordpress/wp-content/uploads/ipc-sm-782a_amendment_1_and_2.pdf)")
 		(tags "capacitor handsolder")
 		(property "Reference" "C1"
-			(at 0 -1.43 90)
+			(at 0 -1.43 0)
 			(layer "F.SilkS")
 			(effects
@@
 		)
 		(property "Value" "1uF"
-			(at 0 1.43 90)
+			(at 0 1.43 0)
 			(layer "F.Fab")
 			(effects
@@
 		)
 		(property "Datasheet" ""
-			(at 0 0 90)
+			(at 0 0 0)
 			(layer "F.Fab")
 			(hide yes)
@@
 		)
 		(property "Description" "Unpolarized capacitor"
-			(at 0 0 90)
+			(at 0 0 0)
 			(layer "F.Fab")
 			(hide yes)
@@
 		)
 		(fp_text user "${REFERENCE}"
-			(at 0 0 90)
+			(at 0 0 0)
 			(layer "F.Fab")
 			(effects
@@
 		)
 		(pad "1" smd roundrect
-			(at -0.8625 0 90)
+			(at -0.8625 0)
 			(size 1.075 0.95)
 			(layers "F.Cu" "F.Mask" "F.Paste")
@@
 		)
 		(pad "2" smd roundrect
-			(at 0.8625 0 90)
+			(at 0.8625 0)
 			(size 1.075 0.95)
 			(layers "F.Cu" "F.Mask" "F.Paste")

Commit message: Рефакторинг. Расстановка "спиц" теперь, вручную
Parts:
- added C63: 100 nF, Capacitor_SMD:C_0402_1005Metric_Pad0.74x0.62mm_HandSolder, F.Cu at (153.5, 101.5)
- C55: value 1uF -> 4.7 uF
- C56, C59, C62: value 100 nF -> 1uF; footprint Capacitor_SMD:C_0402_1005Metric_Pad0.74x0.62mm_HandSolder -> Capacitor_SMD:C_0603_1608Metric_Pad1.08x0.95mm_HandSolder
- C57, C61: value 1uF -> 100 nF; footprint Capacitor_SMD:C_0603_1608Metric_Pad1.08x0.95mm_HandSolder -> Capacitor_SMD:C_0402_1005Metric_Pad0.74x0.62mm_HandSolder
- moved C22 5.98 mm to (160.0, 99.4), turned to 180 degrees
Connections:
- C55 pad 1: +3V3 -> +1V2_VCCD_PLL
- C57 pad 1: +3V3_OSCILL -> +3V3
- C58 pad 1: +3V3 -> +3V3_OSCILL
- C59 pad 1: GND -> +3V3
- C59 pad 2: +3V3_OSCILL -> GND
- C60 pad 1: +3V3 -> GND
- C60 pad 2: GND -> +3V3_OSCILL
- C61 pad 1: +3V3_FLASH -> +3V3
- C62 pad 1: GND -> +3V3_FLASH
- C62 pad 2: +3V3_FLASH -> GND
