File: test_boards/Power/Power.kicad_pcb (KiCad board)
At the start: 4 copper layers, 55 parts, among them J201 ±5V In, U201 AMS1117-1.2, U202 AMS1117CD-3.3, U203 LM317_TO-252, U204 LM337_TO252

Commit message: добавлен общий профиль конфигов
Parts:
- removed C201, C202: TAJD107K016RNJ, Capacitor_Tantalum_SMD:CP_EIA-7343-20_Kemet-V_HandSolder
- removed C203, C204, C211, C212, C215, C216, C217, C218, C219, C220, C225, C226: 100 nF, Capacitor_SMD:C_0603_1608Metric_Pad1.08x0.95mm_HandSolder
- removed C205, C206: TAJB476K010UNJ, Capacitor_Tantalum_SMD:CP_EIA-3528-12_Kemet-T_HandSolder
- removed C207, C208, C209, C210, C213, C214, C221, C222: 1 uF, Capacitor_SMD:C_1206_3216Metric_Pad1.33x1.80mm_HandSolder
- removed C223, C224: 10 uF, Capacitor_SMD:C_1206_3216Metric_Pad1.33x1.80mm_HandSolder
- removed D201, D202, D203, D208, D209: LED, Diode_SMD:D_0805_2012Metric_Pad1.15x1.40mm_HandSolder
- removed D204, D205, D206, D207: D, Diode_SMD:D_SMA_Handsoldering
- removed FB201, FB202: BLM21PG121SN1D, Inductor_SMD:L_0805_2012Metric
- removed FB203, FB204, FB205, FB206: BLM15PD121SN1D, Inductor_SMD:L_0402_1005Metric
- removed J201: ±5V In, Connector_JST:JST_XH_B3B-XH-A_1x03_P2.50mm_Vertical
- removed R203, R204: 470, Resistor_SMD:R_0603_1608Metric_Pad0.98x0.95mm_HandSolder
- removed R205: 330, Resistor_SMD:R_0603_1608Metric_Pad0.98x0.95mm_HandSolder
- removed R206, R207, R208, R209: 240, Resistor_SMD:R_0603_1608Metric_Pad0.98x0.95mm_HandSolder
- removed R210, R211: 220, Resistor_SMD:R_0603_1608Metric_Pad0.98x0.95mm_HandSolder
- removed U201: AMS1117-1.2, Package_TO_SOT_SMD:SOT-223-3_TabPin2
- removed U202: AMS1117CD-3.3, Package_TO_SOT_SMD:TO-252-3_TabPin2
- removed U203: LM317_TO-252, Package_TO_SOT_SMD:TO-252-2
- removed U204: LM337_TO252, Package_TO_SOT_SMD:TO-252-2
- added C1: TAJD107K016RNJ, Capacitor_Tantalum_SMD:CP_EIA-7343-20_Kemet-V_HandSolder, F.Cu at (41.2, 56.3)
- added C10: 1 uF, Capacitor_SMD:C_1206_3216Metric_Pad1.33x1.80mm_HandSolder, F.Cu at (111.2, 72.5)
- added C11: 1 uF, Capacitor_SMD:C_1206_3216Metric_Pad1.33x1.80mm_HandSolder, F.Cu at (111.2, 75.9)
- added C12: 100 nF, Capacitor_SMD:C_0603_1608Metric_Pad1.08x0.95mm_HandSolder, F.Cu at (128.6, 72.9)
- added C13: 1 uF, Capacitor_SMD:C_1206_3216Metric_Pad1.33x1.80mm_HandSolder, F.Cu at (111.2, 79.2)
- added C14: 1 uF, Capacitor_SMD:C_1206_3216Metric_Pad1.33x1.80mm_HandSolder, F.Cu at (111.2, 82.6)
- added C15: 100 nF, Capacitor_SMD:C_0603_1608Metric_Pad1.08x0.95mm_HandSolder, F.Cu at (128.6, 75.5)
- added C16: 100 nF, Capacitor_SMD:C_0603_1608Metric_Pad1.08x0.95mm_HandSolder, F.Cu at (128.6, 78.0)
- added C17: 100 nF, Capacitor_SMD:C_0603_1608Metric_Pad1.08x0.95mm_HandSolder, F.Cu at (128.6, 80.5)
- added C18: 100 nF, Capacitor_SMD:C_0603_1608Metric_Pad1.08x0.95mm_HandSolder, F.Cu at (128.6, 83.0)
- added C19: 100 nF, Capacitor_SMD:C_0603_1608Metric_Pad1.08x0.95mm_HandSolder, F.Cu at (132.9, 65.4)
- added C2: TAJD107K016RNJ, Capacitor_Tantalum_SMD:CP_EIA-7343-20_Kemet-V_HandSolder, F.Cu at (141.6, 93.0)
- added C20: 100 nF, Capacitor_SMD:C_0603_1608Metric_Pad1.08x0.95mm_HandSolder, F.Cu at (132.9, 67.9)
- added C21: 1 uF, Capacitor_SMD:C_1206_3216Metric_Pad1.33x1.80mm_HandSolder, F.Cu at (111.2, 85.9)
- added C22: 1 uF, Capacitor_SMD:C_1206_3216Metric_Pad1.33x1.80mm_HandSolder, F.Cu at (111.2, 89.3)
- added C23: 10 uF, Capacitor_SMD:C_1206_3216Metric_Pad1.33x1.80mm_HandSolder, F.Cu at (111.2, 92.6)
- added C24: 10 uF, Capacitor_SMD:C_1206_3216Metric_Pad1.33x1.80mm_HandSolder, F.Cu at (111.2, 96.0)
- added C25: 100 nF, Capacitor_SMD:C_0603_1608Metric_Pad1.08x0.95mm_HandSolder, F.Cu at (132.9, 70.4)
- added C26: 100 nF, Capacitor_SMD:C_0603_1608Metric_Pad1.08x0.95mm_HandSolder, F.Cu at (132.9, 72.9)
- added C3: 100 nF, Capacitor_SMD:C_0603_1608Metric_Pad1.08x0.95mm_HandSolder, F.Cu at (44.7, 54.0)
- added C4: 100 nF, Capacitor_SMD:C_0603_1608Metric_Pad1.08x0.95mm_HandSolder, F.Cu at (128.6, 67.9)
- added C5: TAJB476K010UNJ, Capacitor_Tantalum_SMD:CP_EIA-3528-12_Kemet-T_HandSolder, F.Cu at (139.7, 98.1)
- added C6: TAJB476K010UNJ, Capacitor_Tantalum_SMD:CP_EIA-3528-12_Kemet-T_HandSolder, F.Cu at (139.7, 102.5)
- added C7: 1 uF, Capacitor_SMD:C_1206_3216Metric_Pad1.33x1.80mm_HandSolder, F.Cu at (47.0, 54.7)
- added C8: 1 uF, Capacitor_SMD:C_1206_3216Metric_Pad1.33x1.80mm_HandSolder, F.Cu at (111.2, 69.2)
- added C9: 100 nF, Capacitor_SMD:C_0603_1608Metric_Pad1.08x0.95mm_HandSolder, F.Cu at (49.2, 54.0)
- added D1: LED, Diode_SMD:D_0805_2012Metric_Pad1.15x1.40mm_HandSolder, F.Cu at (141.9, 65.7)
- added D2: LED, Diode_SMD:D_0805_2012Metric_Pad1.15x1.40mm_HandSolder, F.Cu at (141.9, 68.7)
- added D3: LED, Diode_SMD:D_0805_2012Metric_Pad1.15x1.40mm_HandSolder, F.Cu at (141.9, 71.8)
- added D4: D, Diode_SMD:D_SMA_Handsoldering, F.Cu at (131.5, 86.5)
- added D5: D, Diode_SMD:D_SMA_Handsoldering, F.Cu at (131.5, 91.1)
- added D6: D, Diode_SMD:D_SMA_Handsoldering, F.Cu at (131.5, 95.6)
- added D7: D, Diode_SMD:D_SMA_Handsoldering, F.Cu at (131.5, 100.2)
- added D8: LED, Diode_SMD:D_0805_2012Metric_Pad1.15x1.40mm_HandSolder, F.Cu at (141.9, 74.8)
- added D9: LED, Diode_SMD:D_0805_2012Metric_Pad1.15x1.40mm_HandSolder, F.Cu at (141.9, 77.8)
- added FB1: BLM21PG121SN1D, Inductor_SMD:L_0805_2012Metric, F.Cu at (45.8, 50.6)
- added FB2: BLM21PG121SN1D, Inductor_SMD:L_0805_2012Metric, F.Cu at (110.5, 101.8)
- added FB3: BLM15PD121SN1D, Inductor_SMD:L_0402_1005Metric, F.Cu at (144.3, 96.9)
- added FB4: BLM15PD121SN1D, Inductor_SMD:L_0402_1005Metric, F.Cu at (144.3, 98.9)
- added FB5: BLM15PD121SN1D, Inductor_SMD:L_0402_1005Metric, F.Cu at (144.3, 100.9)
- added FB6: BLM15PD121SN1D, Inductor_SMD:L_0402_1005Metric, F.Cu at (144.3, 102.9)
- added J1: ±5V In, Connector_JST:JST_XH_B3B-XH-A_1x03_P2.50mm_Vertical, F.Cu at (30.5, 48.1)
- added R1: 470, Resistor_SMD:R_0603_1608Metric_Pad0.98x0.95mm_HandSolder, F.Cu at (132.9, 75.5)
- added R2: 470, Resistor_SMD:R_0603_1608Metric_Pad0.98x0.95mm_HandSolder, F.Cu at (132.9, 78.0)
- added R3: 330, Resistor_SMD:R_0603_1608Metric_Pad0.98x0.95mm_HandSolder, F.Cu at (132.9, 80.5)
- added R4: 240, Resistor_SMD:R_0603_1608Metric_Pad0.98x0.95mm_HandSolder, F.Cu at (132.9, 83.0)
- added R5: 240, Resistor_SMD:R_0603_1608Metric_Pad0.98x0.95mm_HandSolder, F.Cu at (137.3, 65.4)
- added R6: 240, Resistor_SMD:R_0603_1608Metric_Pad0.98x0.95mm_HandSolder, F.Cu at (137.3, 67.9)
- added R7: 240, Resistor_SMD:R_0603_1608Metric_Pad0.98x0.95mm_HandSolder, F.Cu at (137.3, 70.4)
- added R8: 220, Resistor_SMD:R_0603_1608Metric_Pad0.98x0.95mm_HandSolder, F.Cu at (137.3, 72.9)
- added R9: 220, Resistor_SMD:R_0603_1608Metric_Pad0.98x0.95mm_HandSolder, F.Cu at (137.3, 75.5)
- added U1: AMS1117-1.2, Package_TO_SOT_SMD:SOT-223-3_TabPin2, F.Cu at (119.2, 100.7)
- added U2: AMS1117CD-3.3, Package_TO_SOT_SMD:TO-252-3_TabPin2, F.Cu at (121.2, 68.3)
- added U3: LM317_TO-252, Package_TO_SOT_SMD:TO-252-2, F.Cu at (121.2, 76.5)
- added U4: LM337_TO252, Package_TO_SOT_SMD:TO-252-2, F.Cu at (121.2, 84.7)
