File: test_boards/Power/Power.kicad_sch (KiCad schematic)
At the start: 55 parts, among them J201 ±5V In, U201 AMS1117-1.2, U202 AMS1117CD-3.3, U203 LM317_TO-252, U204 LM337_TO252

Commit message: добавлен общий профиль конфигов
Parts:
- renumbered C201 to C1, C209 to C10, C210 to C11, C212 to C12, C213 to C13, C214 to C14, C215 to C15, C216 to C16, C217 to C17, C218 to C18, C219 to C19, C202 to C2, C220 to C20, C221 to C21, C222 to C22, C223 to C23, C224 to C24, C225 to C25, C226 to C26, C203 to C3, C204 to C4, C205 to C5, C206 to C6, C207 to C7, C208 to C8, C211 to C9, D201 to D1, D202 to D2, D203 to D3, D204 to D4, D205 to D5, D206 to D6, D207 to D7, D208 to D8, D209 to D9, FB201 to FB1, FB202 to FB2, FB203 to FB3, FB204 to FB4, FB205 to FB5, FB206 to FB6, J201 to J1, R203 to R1, R204 to R2, R205 to R3, R206 to R4, R207 to R5, R208 to R6, R209 to R7, R210 to R8, R211 to R9, U201 to U1, U202 to U2, U203 to U3, U204 to U4
